File: kicad/corone/corone.kicad_sch (KiCad schematic)
At the start: 89 parts, among them J1 To main board, J2 SWD, J3 Debug UART, SW1 BOOT0, SW2 RESET, U1 AMS1117-5.0, U2 AP2112K-3.3, U3 ADS131A02IPBS, U4 DAC8565IAPW, U5 OPA4197, U6 OPA4197, U7 ADG1408YRUZ, U8 STM32F722RET6, U9 USBLC6-2SC6, Y1 8MHz

Commit message: Corone header: swap pins 17 and 18 (GND on 17, USB VBUS sense on 18)
Both sides of the 2x10: J121 on the main board, J1 on Corone, and the
pinout in corone/README.md. For routing; electrically the same.

Co-Authored-By: Claude Opus 5.5 <noreply@anthropic.com>
Connections:
- net GND: now also J1.17 (Pin_17); no longer J1.18 (Pin_18)
- net VBUS: now also J1.18 (Pin_18); no longer J1.17 (Pin_17)
Changed lines of the file:
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@@
-		)
-	)
-	(label "VBUS"
-		(at 40.64 73.66 180)
-		(effects
-			(font
-				(size 1.27 1.27)
-			)
-			(justify right bottom)
 		)
 	)
 	(symbol
 		(lib_id "power:GND")
-		(at 53.34 73.66 0)
+		(at 40.64 73.66 0)
 		(unit 1)
 		(exclude_from_sim no)
@@
 		(dnp no)
 		(property "Reference" "#PWR008"
-			(at 55.88 66.04 0)
+			(at 43.18 66.04 0)
 			(hide yes)
 			(effects
@@
 		)
 		(property "Value" "GND"
-			(at 55.88 81.28 0)
+			(at 43.18 81.28 0)
 			(effects
 				(font
@@
 		)
 		(property "Footprint" ""
-			(at 53.34 73.66 0)
+			(at 40.64 73.66 0)
 			(hide yes)
 			(effects
@@
 		)
 		(property "Datasheet" ""
-			(at 53.34 73.66 0)
+			(at 40.64 73.66 0)
 			(hide yes)
 			(effects
@@
 		)
 	)
+	(label "VBUS"
+		(at 53.34 73.66 0)
+		(effects
+			(font
+				(size 1.27 1.27)
+			)
+			(justify left bottom)
+		)
+	)
