File: kicad/corone/corone.kicad_pcb (KiCad board)
At the start: 2 copper layers, 63.3 x 49.8 mm, 91 parts, among them J1 To main board, J2 SWD, J3 Debug UART, SW1 BOOT0, SW2 RESET, U1 AMS1117-5.0, U2 AP2112K-3.3, U3 ADS131A02IPBS, U4 DAC8565IAPW, U5 OPA4197, U6 OPA4197, U7 ADG1408YRUZ, U8 STM32F722RET6, U9 USBLC6-2SC6, Y1 8MHz

Commit message: MIDI out A/B: 2 x 3 header and shunts (J123) in place of the solder jumpers
Odd pins the tip, even the ring, the middle row the jack: both shunts on
the top row is Type A, on the bottom row Type B. J123 keeps JP101's
symbol id, so the board links without Update PCB; its tracks are left to
route. Also takes in the board edits saved since the last commit.

Co-Authored-By: Claude Opus 5.5 <noreply@anthropic.com>
Changed lines of the file:
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@@
 		(tags "resistor")
 		(property "Reference" "R11"
-			(at 0 -1.43 0)
+			(at -2.85 0.1 0)
 			(layer "F.SilkS")
 			(effects
@@
 		(tags "LQFP QFP")
 		(property "Reference" "U8"
-			(at 0 -7.4 0)
+			(at -0.2 -0.325 0)
 			(layer "F.SilkS")
 			(effects
@@
 		(tags "capacitor")
 		(property "Reference" "C51"
-			(at 0 -1.43 90)
+			(at -2.75 -0.15 90)
 			(layer "F.SilkS")
 			(effects
@@
 		(tags "capacitor")
 		(property "Reference" "C2"
-			(at 0 -1.68 90)
+			(at 1.2 -1.45 90)
 			(layer "F.SilkS")
 			(effects
@@
 		(tags "resistor")
 		(property "Reference" "R64"
-			(at 0 -1.43 0)
+			(at 2.05 0.1 90)
 			(layer "F.SilkS")
 			(effects
@@
 		(tags "TSSOP SO JEDEC-MO-153-AB Texas_PW0016A Microchip-ST Toshiba-TSSOP16-P-0044-0.65A NXP-SOT403-1 Infineon-P-TSSOP-16-800")
 		(property "Reference" "U4"
-			(at 0 -3.45 90)
+			(at 0.0625 -0.025 90)
 			(layer "F.SilkS")
 			(effects
@@
 		(tags "resistor")
 		(property "Reference" "R56"
-			(at 0 -1.43 0)
+			(at 0.075 1.35 0)
 			(layer "F.SilkS")
 			(effects
@@
 		(tags "SOT TO_SOT_SMD")
 		(property "Reference" "U9"
-			(at 0 -2.4 0)
+			(at 0.0625 2.25 0)
 			(layer "F.SilkS")
 			(effects
@@
 		(tags "TSSOP SO")
 		(property "Reference" "U6"
-			(at 0 -3.45 90)
+			(at -0.0125 -0.075 90)
 			(layer "F.SilkS")
 			(effects
@@
 		(tags "capacitor")
 		(property "Reference" "C5"
-			(at 0.075 -1.708571 90)
+			(at -2.9 0.2 90)
 			(layer "F.SilkS")
 			(effects
@@
 		(tags "capacitor")
 		(property "Reference" "C1"
-			(at 0 -1.68 0)
+			(at -0.725 -1.45 0)
 			(layer "F.SilkS")
 			(effects
@@
 		(tags "SOT TO_SOT_SMD")
 		(property "Reference" "U2"
-			(at 0 -2.4 90)
+			(at 0.0875 2.15 90)
 			(layer "F.SilkS")
 			(effects
@@
 	)
 	(footprint "Connector_PinHeader_2.54mm:PinHeader_1x03_P2.54mm_Vertical"
+		(locked yes)
 		(layer "F.Cu")
 		(at 141.04 105.95 -90)
@@
 		(tags "capacitor")
 		(property "Reference" "C4"
-			(at 0 -1.68 90)
+			(at 0.015001 1.8 90)
 			(layer "F.SilkS")
 			(effects
@@
 		)
 		(property "Value" "To main board"
-			(at -1.27 -25.63 180)
+			(at -5.339999 -17.6 90)
 			(layer "B.Fab")
 			(effects
