File: kicad/shieldXL-euro/eurorack.kicad_sch (KiCad schematic)
At the start: 62 parts, among them J101 Eurorack power, J102 IN L, J103 IN R, J104 OUT L, J105 OUT R, J106 MIDI IN, J107 MIDI OUT, J108 DX07S024WJ1R350, J109 USB 1, J110 USB 2, J111 USB 3, J112 Pi USB, inner stack, J113 Pi USB, outer stack, J115 CORONE I/1, J116 CORONE I/2, J117 CORONE O/1, J118 CORONE O/2, J119 CORONE O/3, J120 CORONE O/4, J121 Corone, J122 ii, J123 MIDI OUT A/B, U101 TL074, U102 USBLC6-2SC6, U103 USBLC6-2SC6, U104 USBLC6-2SC6, U105 74LVC1G125

Commit message: Codec: TI PCM3060 in place of the end-of-life CS4270
U1 swaps in place on the shield sheet (tools/swap_codec_pcm3060.py, pin
map there): same wires, same uuid, so Update PCB brings in the TSSOP-28.
I2C at 0x46 (MODE and ADR low); ADC and DAC share the clocks; the codec
stays clock master off the 12.288 MHz crystal, the DAC driving BCK/LRCK
and the ADC following. FILT+ caps C6/C7 off the board.

Levels re-set for the PCM3060 at 4.75 V: input divider 1.27k / 4.53k into
its 10k input (13.3 Vpp full scale), output gain 2.62 (R106/R109 16.2k)
for 10 Vpp from its 3.8 Vpp single-ended DAC.

Software: the kernel's pcm3060 driver with one DT flag so the ADC stays a
clock consumer (software/pcm3060-moirae), and a norns overlay
(install/boot/overlays/moirae-pcm3060-overlay.dts). Untested on hardware.

Co-Authored-By: Claude Opus 5.5 <noreply@anthropic.com>
Parts:
- R106, R109: value 24.9k -> 16.2k
Changed lines of the file:
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@@
 			)
 		)
-		(property "Value" "24.9k"
+		(property "Value" "16.2k"
 			(at 167.64 101.6 0)
 			(effects
@@
 			)
 		)
-		(property "Value" "24.9k"
+		(property "Value" "16.2k"
 			(at 167.64 132.08 0)
 			(effects
