File: kicad/shieldXL-euro/norns-shield-210330_1.kicad_sch (KiCad schematic)
At the start: 39 parts, among them Q1 ASFL1-12.288MHZ-LCS-T, U1 CS4270, U11 TPS793475DBVR, X1 RASPI_BOARD_B+#_E3

Commit message: Pi: screw down only the two holes by the header
The other two fall on K1's and E2's pins; those corners stand on
3D-printed feet fixed to the Pi. New footprint MMM:RASPI_BOARD_B+_UPPER_HOLES
for X1, the feet drawn on User.3.

Co-Authored-By: Claude Opus 5.5 <noreply@anthropic.com>
Parts:
- X1: footprint ShieldXL:RASPI_BOARD_B+_EDGES_3DRILL -> MMM:RASPI_BOARD_B+_UPPER_HOLES
Changed lines of the file:
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@@
 			)
 		)
-		(property "Footprint" "ShieldXL:RASPI_BOARD_B+_EDGES_3DRILL"
+		(property "Footprint" "MMM:RASPI_BOARD_B+_UPPER_HOLES"
 			(at 114.3 166.37 0)
 			(effects

Commit message: Pi stack in 3D: 20 mm, socket plus stacking header
X1 carries three models: the Pi, hung 20 mm behind the board's back so its
USB stacks (16 mm) clear the SMD parts under them by 2 mm, and two 2x20
socket bodies standing in for an 8.5 mm socket on the board with a stacking
header in it. X1 is populated now (the socket is fitted to the board), so it
shows in renders and exports.

Co-Authored-By: Claude Opus 5.5 <noreply@anthropic.com>
Parts:
- X1: now fitted
Changed lines of the file:
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@@
 		(in_bom yes)
 		(on_board yes)
-		(dnp yes)
+		(dnp no)
 		(property "Reference" "X1"
 			(at 114.3 124.46 0)

Commit message: Codec: TI PCM3060 in place of the end-of-life CS4270
U1 swaps in place on the shield sheet (tools/swap_codec_pcm3060.py, pin
map there): same wires, same uuid, so Update PCB brings in the TSSOP-28.
I2C at 0x46 (MODE and ADR low); ADC and DAC share the clocks; the codec
stays clock master off the 12.288 MHz crystal, the DAC driving BCK/LRCK
and the ADC following. FILT+ caps C6/C7 off the board.

Levels re-set for the PCM3060 at 4.75 V: input divider 1.27k / 4.53k into
its 10k input (13.3 Vpp full scale), output gain 2.62 (R106/R109 16.2k)
for 10 Vpp from its 3.8 Vpp single-ended DAC.

Software: the kernel's pcm3060 driver with one DT flag so the ADC stays a
clock consumer (software/pcm3060-moirae), and a norns overlay
(install/boot/overlays/moirae-pcm3060-overlay.dts). Untested on hardware.

Co-Authored-By: Claude Opus 5.5 <noreply@anthropic.com>
Parts:
- C6, C7: now not fitted; now left out of the parts list
- R10, R8: value 10k -> 4.53k
- R7, R9: value 4.99k -> 1.27k
- U1: value CS4270 -> PCM3060PW; footprint ShieldXL:TSSOP24 -> Package_SO:TSSOP-28_4.4x9.7mm_P0.65mm; symbol norns-shield-210330-eagle-import:CS4270 -> Moirae:PCM3060
Connections:
- net +3V3: now also U1.7 (VDD); no longer U1.5 (VD), U1.8 (VLC)
- net A5V: now also U1.24 (VCC); no longer U1.19 (VA)
- net AGND: now also U1.16 (SGND), U1.22 (AGND2), U1.23 (AGND1); no longer U1.20 (AGND)
- net GND: now also U1.27 (MS/ADR), U1.28 (MODE), U1.8 (DGND); no longer U1.11 (CS), U1.12 (CDIN), U1.13 (AD2), U1.6 (DGND)
- net INA: now also U1.26 (VINR); no longer U1.16 (AINB)
- net INB: now also U1.25 (VINL); no longer U1.15 (AINA)
- net LRCK: now also U1.11 (LRCK2), U1.4 (LRCK1); no longer U1.2 (LRCK)
- net MCLK: now also U1.6 (SCKI1), U1.9 (SCKI2); no longer U1.3 (MCLK)
- net OUTA: now also U1.18 (VOUTR+); no longer U1.23 (AOUTB)
- net OUTB: now also U1.20 (VOUTL+); no longer U1.22 (AOUTA)
- net R-CODEC: now also U1.15 (~{RST}); no longer U1.14 (_RST)
- net SCL: now also U1.1 (MC/SCL); no longer U1.10 (CCLK)
- net SCLK: now also U1.10 (BCK2), U1.5 (BCK1); no longer U1.4 (SCLK)
- net SDA: now also U1.2 (MD/SDA); no longer U1.9 (CDOUT)
- net SDIN: now also U1.12 (DIN); no longer U1.1 (SDIN)
- net SDOUT: now also U1.3 (DOUT); no longer U1.7 (SDOUT)
- net at C4.1, C5.1: now also U1.21 (VCOM); no longer U1.17 (VQ)
- net at C6.1, C7.1: no longer U1.18 (FILT+)
- no-connect marks 0 -> 4
Changed lines of the file:
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@@
 		(color 0 0 0 0)
 	)
+	(no_connect
+		(at 259.08 99.06)
+	)
+	(no_connect
+		(at 259.08 91.44)
+	)
+	(no_connect
+		(at 248.92 81.28)
+	)
+	(no_connect
+		(at 251.46 81.28)
+	)
 	(wire
 		(pts
@@
 	(wire
 		(pts
-			(xy 213.36 109.22) (xy 182.88 109.22)
-		)
-		(stroke
-			(width 0.1524)
-			(type solid)
-		)
-	)
-	(wire
-		(pts
 			(xy 259.08 104.14) (xy 294.64 104.14)
 		)
@@
 	(wire
 		(pts
-			(xy 259.08 106.68) (xy 279.4 106.68)
-		)
-		(stroke
-			(width 0.1524)
-			(type solid)
-		)
-	)
-	(wire
-		(pts
 			(xy 365.76 167.64) (xy 373.38 167.64)
 		)
@@
 	(wire
 		(pts
-			(xy 279.4 106.68) (xy 279.4 119.38)
-		)
-		(stroke
-			(width 0.1524)
-			(type solid)
-		)
-	)
-	(wire
-		(pts
 			(xy 137.16 193.04) (xy 137.16 190.5)
 		)
@@
 	(wire
 		(pts
-			(xy 259.08 121.92) (xy 259.08 119.38)
-		)
-		(stroke
-			(width 0.1524)
-			(type solid)
-		)
-	)
-	(wire
-		(pts
 			(xy 205.74 180.34) (xy 205.74 177.8)
 		)
@@
 	(wire
 		(pts
-			(xy 182.88 109.22) (xy 182.88 101.6)
-		)
-		(stroke
-			(width 0.1524)
-			(type solid)
-		)
-	)
-	(wire
-		(pts
 			(xy 91.44 157.48) (xy 99.06 157.48)
 		)
@@
 			)
 		)
-		(property "Value" "4.99k"
+		(property "Value" "1.27k"
 			(at 133.35 187.198 0)
 			(effects
@@
 		(unit 1)
 		(exclude_from_sim no)
-		(in_bom yes)
-		(on_board yes)
-		(dnp no)
+		(in_bom no)
+		(on_board no)
+		(dnp yes)
 		(property "Reference" "C7"
 			(at 288.036 123.825 0)
@@
 			)
 		)
-		(property "Value" "10k"
+		(property "Value" "4.53k"
 			(at 133.858 222.25 0)
 			(effects
@@
 	)
 	(symbol
-		(lib_id "norns-shield-210330-eagle-import:CS4270")
+		(lib_id "Moirae:PCM3060")
 		(at 236.22 104.14 0)
 		(unit 1)
@@
 			)
 		)
-		(property "Value" "CS4270"
+		(property "Value" "PCM3060PW"
 			(at 243.84 124.46 0)
 			(effects
@@
 			)
 		)
-		(property "Footprint" "ShieldXL:TSSOP24"
+		(property "Footprint" "Package_SO:TSSOP-28_4.4x9.7mm_P0.65mm"
 			(at 236.22 104.14 0)
 			(effects
@@
 			)
 		)
-		(property "Datasheet" ""
+		(property "Datasheet" "https://www.ti.com/lit/ds/symlink/pcm3060.pdf"
 			(at 236.22 104.14 0)
 			(effects
@@
 			)
 		)
-		(pin "1"
+		(pin "12"
 		)
-		(pin "10"
+		(pin "4"
 		)
 		(pin "11"
 		)
-		(pin "12"
-		)
-		(pin "13"
+		(pin "6"
 		)
-		(pin "14"
+		(pin "9"
 		)
-		(pin "15"
+		(pin "5"
 		)
-		(pin "16"
+		(pin "10"
 		)
-		(pin "17"
+		(pin "7"
 		)
-		(pin "18"
+		(pin "8"
 		)
-		(pin "19"
+		(pin "3"
 		)
 		(pin "2"
 		)
-		(pin "20"
+		(pin "1"
+		)
+		(pin "28"
+		)
+		(pin "27"
+		)
+		(pin "15"
+		)
+		(pin "25"
+		)
+		(pin "26"
 		)
 		(pin "21"
 		)
-		(pin "22"
+		(pin "24"
 		)
 		(pin "23"
 		)
-		(pin "24"
+		(pin "22"
 		)
-		(pin "3"
+		(pin "16"
 		)
-		(pin "4"
+		(pin "14"
 		)
-		(pin "5"
+		(pin "20"
 		)
-		(pin "6"
+		(pin "18"
 		)
-		(pin "7"
+		(pin "13"
 		)
-		(pin "8"
+		(pin "19"
 		)
-		(pin "9"
+		(pin "17"
 		)
 		(instances
@@
 	)
 	(symbol
-		(lib_id "norns-shield-210330-eagle-import:GND")
-		(at 259.08 124.46 0)
-		(unit 1)
-		(exclude_from_sim no)
-		(in_bom yes)
-		(on_board yes)
-		(dnp no)
-		(property "Reference" "#GND07"
-			(at 259.08 124.46 0)
-			(effects
-				(font
-					(size 1.27 1.27)
-				)
-				(hide yes)
-			)
-		)
-		(property "Value" "GND"
-			(at 256.54 127 0)
-			(effects
-				(font
-					(size 1.778 1.5113)
-				)
-				(justify left bottom)
-			)
-		)
-		(property "Footprint" ""
-			(at 259.08 124.46 0)
-			(effects
-				(font
-					(size 1.27 1.27)
-				)
-				(hide yes)
-			)
-		)
-		(property "Datasheet" ""
-			(at 259.08 124.46 0)
-			(effects
-				(font
-					(size 1.27 1.27)
-				)
-				(hide yes)
-			)
-		)
-		(property "Description" ""
-			(at 259.08 124.46 0)
-			(effects
-				(font
-					(size 1.27 1.27)
-				)
-				(hide yes)
-			)
-		)
-		(pin "1"
-		)
-		(instances
-			(project "shieldXL-euro"
-				(path "/b86e8947-58dc-49c6-bb5d-ce6d33c2e465/d872c92c-5229-43e6-807a-8bd0f3dfa8f7"
-					(reference "#GND07")
-					(unit 1)
-				)
-			)
-		)
-	)
-	(symbol
 		(lib_id "norns-shield-210330-eagle-import:C-USC0603")
 		(at 330.2 180.34 0)
@@
 			)
 		)
-		(property "Value" "10k"
+		(property "Value" "4.53k"
 			(at 133.858 194.31 0)
 			(effects
@@
 			)
 		)
-		(property "Value" "4.99k"
+		(property "Value" "1.27k"
 			(at 133.35 215.138 0)
 			(effects
@@
 		(unit 1)
 		(exclude_from_sim no)
-		(in_bom yes)
-		(on_board yes)
-		(dnp no)
+		(in_bom no)
+		(on_board no)
+		(dnp yes)
 		(property "Reference" "C6"
 			(at 280.416 123.825 0)
